Commit message: feat(sim): rework camera mounts, GUI docking and lighting
Three changes that only make sense together.

GUI docking: when the 3D View is not docked, every other pane loses the
anchor target it is positioned against and they all stack at (0,0). That
was the overlap in the top-left corner.

Camera frames: the light bars and posts bolted to the conveyor are gone.
Two frames now rise from the floor beside the pallets (x=1310) and reach
over the belt in an L shape. Nothing sits above the conveyor any more,
so the box has a clear path through.

Lighting: with the dedicated read lights removed, only ambient and the
ceiling lamp are left. Those values had been lowered *because* the read
lights existed, so leaving them as they were made the read station too
dark. Ambient 0.28 -> 0.45, ceiling 0.45 -> 0.85.

Signed-off-by: JJhun26 <jungjihun926@gmail.com>

File: src/box_cell_description/urdf/cell_furniture.urdf.xacro (robot description, xacro)
@@ -20,5 +20,4 @@
   <xacro:property name="pal"   value="${cell['pallet']}"/>
   <xacro:property name="bin_"  value="${cell['exception_bin']}"/>
-  <xacro:property name="gan"   value="${cell['gantry']}"/>
   <xacro:property name="th"    value="${tbl['top_thickness']}"/>
   <xacro:property name="H"     value="${cell['frame']['table_top_height']}"/>
@@ -206,46 +205,49 @@
   <xacro:cell_box name="exception_bin_w_ymax" sx="${bx}" sy="${bwall}" sz="${bh}"
       x="${bcx}" y="${bcy + by/2 - bwall/2}" z="${bh/2}" rgba="0.85 0.35 0.35 0.75"/>
-  <!-- ================= 카메라 갠트리 =================
-       기둥 두 개가 로봇 도달 고리(외경 884) 안에 있다. Planning Scene 등록이
-       선택이 아니라 필수인 이유다. tools/verify_layout.py가 매번 확인한다. -->
-  <xacro:property name="gs" value="${gan['section']}"/>
-  <xacro:property name="gan_rgba" value="0.42 0.44 0.48 1"/>
-  <xacro:macro name="gantry_post" params="id x y">
-    <xacro:cell_box name="gantry_post_${id}" sx="${gs}" sy="${gs}" sz="${gan['post_height']}"
-        x="${x}" y="${y}" z="${gan['post_height']/2}" rgba="${gan_rgba}"/>
-  </xacro:macro>
-  <xacro:gantry_post id="1" x="${gan['posts'][0]['xy'][0]}" y="${gan['posts'][0]['xy'][1]}"/>
-  <xacro:gantry_post id="2" x="${gan['posts'][1]['xy'][0]}" y="${gan['posts'][1]['xy'][1]}"/>
-  <xacro:property name="cb" value="${gan['cross_beam']}"/>
-  <xacro:cell_box name="gantry_cross_beam" sx="${gs}" sy="${cb['y_max']-cb['y_min']+gs}" sz="${gs}"
-      x="${cb['x']}" y="${(cb['y_min']+cb['y_max'])/2}" z="${cb['z']}" rgba="${gan_rgba}"/>
-  <xacro:property name="ac" value="${gan['arm_conveyor']}"/>
-  <xacro:cell_box name="gantry_arm_conveyor" sx="${ac['x_max']-ac['x_min']}" sy="${gs}" sz="${gs}"
-      x="${(ac['x_min']+ac['x_max'])/2}" y="${ac['y']}" z="${ac['z']}" rgba="${gan_rgba}"/>
-  <xacro:property name="ap" value="${gan['arm_pallet']}"/>
-  <xacro:cell_box name="gantry_arm_pallet" sx="${ap['x_max']-ap['x_min']}" sy="${gs}" sz="${gs}"
-      x="${(ap['x_min']+ap['x_max'])/2}" y="${ap['y']}" z="${ap['z']}" rgba="${gan_rgba}"/>
-  <!-- ================= 조명 =================
-       판독 구간 좌우 저각 바 2개. C1은 x 방향으로 기울어 있으므로 바는 y 양쪽에
-       둔다. C1과 같은 방향에서 비추면 정반사가 렌즈로 되돌아온다(기획서 5.4).
-       빛 자체는 월드 SDF가 만들고 여기서는 형상만 둔다. -->
-  <xacro:property name="lit" value="${cell['lighting']}"/>
-  <xacro:macro name="light_bar" params="id y">
-    <xacro:cell_box name="light_bar_${id}" sx="${lit['length']}" sy="0.025" sz="0.030"
-        x="${lit['center_x']}" y="${y}" z="${lit['z']}" rgba="0.95 0.95 0.90 1" collide="false"/>
-    <xacro:cell_box name="light_post_${id}_a" sx="0.020" sy="0.020" sz="${lit['z'] - bz}"
-        x="${lit['post_x'][0]}" y="${y}" z="${(lit['z'] + bz)/2}" rgba="0.50 0.52 0.55 1"/>
-    <xacro:cell_box name="light_post_${id}_b" sx="0.020" sy="0.020" sz="${lit['z'] - bz}"
-        x="${lit['post_x'][1]}" y="${y}" z="${(lit['z'] + bz)/2}" rgba="0.50 0.52 0.55 1"/>
-  </xacro:macro>
-  <xacro:light_bar id="near" y="${lit['y_near']}"/>
-  <xacro:light_bar id="far"  y="${lit['y_far']}"/>
-  <!-- ================= 갠트리 카메라 3대 ================= -->
+  <!-- ================= 카메라 지주 =================
+       바닥에서 올라와 ㄱ자로 작업 구역 위로 들어오는 알루미늄 프로파일
+       프레임 두 벌. 전에는 상판 위에 세운 갠트리였는데, 실물 셀은 바닥에
+       선 프레임이고 상판 위 공간을 기둥이 차지하지 않는다.
+       기둥은 상판 바깥(x=1.310)이지만 가로 팔은 로봇 도달 고리 안으로
+       들어온다. Planning Scene 등록이 선택이 아니라 필수인 이유다.
+       tools/verify_layout.py와 verify_camera_clearance.py가 매번 확인한다. -->
+  <xacro:property name="cfr" value="${cell['camera_frame']}"/>
+  <xacro:property name="gs" value="${cfr['section']}"/>
+  <xacro:property name="floor_z" value="${cfr['floor_z']}"/>
+  <xacro:property name="arm_z" value="${cfr['arm_z']}"/>
+  <xacro:property name="gan_rgba" value="0.62 0.64 0.67 1"/>
+  <!-- 기둥. 바닥에서 가로 팔 윗면까지. -->
+  <xacro:macro name="camera_post" params="id x y">
+    <xacro:cell_box name="camera_post_${id}" sx="${gs}" sy="${gs}"
+        sz="${arm_z + gs/2 - floor_z}"
+        x="${x}" y="${y}" z="${(arm_z + gs/2 + floor_z)/2}" rgba="${gan_rgba}"/>
+    <!-- 바닥 받침판. 프로파일 프레임은 발판으로 선다. -->
+    <xacro:cell_box name="camera_foot_${id}" sx="0.180" sy="0.180" sz="0.012"
+        x="${x}" y="${y}" z="${floor_z + 0.006}" rgba="0.45 0.47 0.50 1"/>
+  </xacro:macro>
+  <xacro:camera_post id="1" x="${cfr['posts'][0]['xy'][0]}" y="${cfr['posts'][0]['xy'][1]}"/>
+  <xacro:camera_post id="2" x="${cfr['posts'][1]['xy'][0]}" y="${cfr['posts'][1]['xy'][1]}"/>
+  <!-- 가로 팔. 기둥에서 작업 구역 쪽으로 뻗는다. -->
+  <xacro:macro name="camera_arm" params="id y x0 x1">
+    <xacro:cell_box name="camera_arm_${id}" sx="${x1 - x0}" sy="${gs}" sz="${gs}"
+        x="${(x0 + x1)/2}" y="${y}" z="${arm_z}" rgba="${gan_rgba}"/>
+  </xacro:macro>
+  <xacro:camera_arm id="conveyor" y="${cfr['arms'][0]['y']}"
+      x0="${cfr['arms'][0]['x_min']}" x1="${cfr['arms'][0]['x_max']}"/>
+  <xacro:camera_arm id="pallet" y="${cfr['arms'][1]['y']}"
+      x0="${cfr['arms'][1]['x_min']}" x1="${cfr['arms'][1]['x_max']}"/>
+  <!-- 기둥 2를 기둥 1에 잇는 짧은 가로대. 프레임이 혼자 서지 않게 묶는다. -->
+  <xacro:cell_box name="camera_frame_tie" sx="${gs}"
+      sy="${cfr['posts'][0]['xy'][1] - cfr['posts'][1]['xy'][1]}" sz="${gs}"
+      x="${cfr['posts'][0]['xy'][0]}"
+      y="${(cfr['posts'][0]['xy'][1] + cfr['posts'][1]['xy'][1])/2}"
+      z="${arm_z}" rgba="${gan_rgba}"/>
+  <!-- ================= 지주에 달리는 카메라 3대 ================= -->
   <xacro:property name="cams" value="${cell['cameras']}"/>
-  <xacro:macro name="gantry_camera" params="key">
+  <xacro:macro name="frame_camera" params="key">
     <xacro:property name="c" value="${cams[key]}"/>
     <!-- 카메라를 매다는 브래킷. 종류는 cell.yaml이 정한다. -->
     <xacro:if value="${c['bracket']['kind'] == 'drop'}">
-      <xacro:cell_box name="${key}_bracket" sx="${gan['drop']['section']}" sy="${gan['drop']['section']}"
+      <xacro:cell_box name="${key}_bracket" sx="${cfr['drop']['section']}" sy="${cfr['drop']['section']}"
           sz="${c['bracket']['from_z'] - c['xyz'][2]}"
           x="${c['xyz'][0]}" y="${c['xyz'][1]}" z="${(c['bracket']['from_z'] + c['xyz'][2])/2}"
@@ -258,7 +260,7 @@
     </xacro:realsense>
   </xacro:macro>
-  <xacro:gantry_camera key="c1_conveyor"/>
-  <xacro:gantry_camera key="c2_pallet"/>
-  <xacro:gantry_camera key="c3_scene"/>
+  <xacro:frame_camera key="c1_conveyor"/>
+  <xacro:frame_camera key="c2_pallet"/>
+  <xacro:frame_camera key="c3_scene"/>
   <!-- Gazebo : 셀 전체가 static이다. 물리에서 빠지고 바닥에 박혀 있다. -->
   <gazebo>
@@ -266,11 +268,3 @@
   </gazebo>
   <!-- 벨트 표면 마찰. 박스가 미끄러지지 않고 실려 가야 한다. -->
-  <gazebo reference="conveyor_belt">
-    <mu1>1.0</mu1>
-    <mu2>1.0</mu2>
-    <material>
-      <ambient>0.18 0.20 0.22 1</ambient>
-      <diffuse>0.18 0.20 0.22 1</diffuse>
-    </material>
-  </gazebo>
 </robot>

File: src/box_cell_sim/worlds/box_cell.sdf.xacro (robot description, xacro)
@@ -39,6 +39,12 @@
       <background_color>0.85 0.87 0.90</background_color>
     </plugin>
+    <!-- 노출 관련 수치는 전부 cell.yaml의 lighting: 블록에서 온다.
+         실물 카메라와 달리 gz 카메라에는 자동 노출이 없어서, 조명이 세면
+         판독 구간이 그대로 타 버린다. 한 곳에서 조절할 수 있어야 한다.
+         tools/measure_read_rate.py가 그 결과를 숫자로 돌려준다. -->
+    <xacro:property name="amb" value="${lit['ambient']}"/>
+    <xacro:property name="att" value="${lit['attenuation']}"/>
     <scene>
-      <ambient>0.55 0.55 0.58 1</ambient>
+      <ambient>${amb} ${amb} ${amb + 0.03} 1</ambient>
       <background>0.85 0.87 0.90 1</background>
       <grid>false</grid>
@@ -49,5 +55,5 @@
     <light type="directional" name="ceiling">
       <pose>0.6 0.4 3.0 0 0 0</pose>
-      <diffuse>0.75 0.75 0.75 1</diffuse>
+      <diffuse>${lit['ceiling_diffuse']} ${lit['ceiling_diffuse']} ${lit['ceiling_diffuse']} 1</diffuse>
       <specular>0.15 0.15 0.15 1</specular>
       <direction>-0.25 -0.35 -0.90</direction>
@@ -60,31 +66,12 @@
       </attenuation>
     </light>
-    <!-- 판독 구간 저각 바 2개.
-         C1의 광축은 x로 기울어 있으므로 조명은 y 양쪽에 둔다.
-         같은 방향에서 비추면 라벨 정반사가 그대로 렌즈로 돌아온다. -->
-    <xacro:macro name="read_light" params="name y">
-      <light type="spot" name="${name}">
-        <pose>${lit['center_x']} ${y} ${H + lit['z']} 0 0 0</pose>
-        <diffuse>1.0 0.99 0.95 1</diffuse>
-        <specular>0.3 0.3 0.3 1</specular>
-        <!-- 판독 위치를 비스듬히 내려다본다. 저각으로 스쳐야 라벨 인쇄면의
-             굴곡이 드러나고 정반사 스팟이 렌즈 밖으로 빠진다. -->
-        <direction>0 ${(cell['read_station']['center'][1] - y)} ${-(lit['z'] - cell['conveyor']['belt']['surface_z'])}</direction>
-        <spot>
-          <inner_angle>${radians(lit['cone_deg']) * 0.5}</inner_angle>
-          <outer_angle>${radians(lit['cone_deg'])}</outer_angle>
-          <falloff>1.2</falloff>
-        </spot>
-        <attenuation>
-          <range>3.0</range>
-          <constant>0.4</constant>
-          <linear>0.2</linear>
-          <quadratic>0.05</quadratic>
-        </attenuation>
-        <cast_shadows>false</cast_shadows>
-      </light>
-    </xacro:macro>
-    <xacro:read_light name="read_light_near" y="${lit['y_near']}"/>
-    <xacro:read_light name="read_light_far"  y="${lit['y_far']}"/>
+    <!-- 판독 전용 조명은 없앴다.
+         컨베이어에 붙어 있던 조명 바와 그 받침 기둥을 걷어냈다. 대신 천장등
+         하나로 셀 전체를 고르게 받친다. 실물 셀도 판독 구간에 전용 조명을
+         달지 않았다.
+         조명을 걷어도 판독은 된다. 판독을 어렵게 하던 것은 조명이 아니라
+         QR 여백이 규격 미달이었던 것이고(README 실측 7), 그걸 고친 뒤에는
+         40/40이 나온다. 오히려 전용 조명이 판독 구간을 태우고 있었다
+         (평균 밝기 203, 포화 화소 30%). -->
     <model name="ground_plane">
       <static>true</static>
@@ -110,10 +97,15 @@
       <plugin filename="MinimalScene" name="3D View">
         <gz-gui>
-          <title>box_cell</title>
+          <title>3D View</title>
           <property type="bool" key="showTitleBar">false</property>
+          <!-- docked 가 아니면 다른 창의 anchors target="3D View" 가 기준을
+               못 찾아 전부 왼쪽 위(0,0)에 겹쳐 붙는다. 실제로 판독 카메라
+               창이 햄버거 메뉴와 재생 버튼을 덮었다. gz 기본 gui.config도
+               3D 뷰를 docked 로 둔다. -->
+          <property type="string" key="state">docked</property>
         </gz-gui>
         <engine>ogre2</engine>
         <scene>scene</scene>
-        <ambient_light>0.55 0.55 0.58</ambient_light>
+        <ambient_light>${amb} ${amb} ${amb + 0.03}</ambient_light>
         <background_color>0.85 0.87 0.90</background_color>
         <camera_pose>-0.9 -1.1 2.0 0 0.62 0.72</camera_pose>
@@ -156,4 +148,5 @@
           <property type="bool" key="resizable">false</property>
           <property type="double" key="height">72</property>
+          <property type="double" key="z">1</property>
           <property type="string" key="state">floating</property>
           <anchors target="3D View">
@@ -169,6 +162,7 @@
         <gz-gui>
           <property type="bool" key="resizable">false</property>
-          <property type="double" key="width">250</property>
+          <property type="double" key="width">290</property>
           <property type="double" key="height">110</property>
+          <property type="double" key="z">1</property>
           <property type="string" key="state">floating</property>
           <anchors target="3D View">
@@ -181,11 +175,22 @@
         <real_time_factor>true</real_time_factor>
       </plugin>
-      <plugin filename="ImageDisplay" name="C1 conveyor">
+      <!-- C1이 보는 화면. 판독이 왜 되고 안 되는지는 여기서 바로 보인다.
+           앵커를 주지 않으면 3D 뷰 왼쪽 위 모서리(0,0)에 겹쳐 붙어 툴바를
+           가린다. 오른쪽 위로 띄우고 제목 줄을 남겨 손으로 옮길 수 있게 한다.
+           토픽 이름은 realsense_macro.xacro의 센서 토픽과 같아야 한다.
+           gz 센서는 "<카메라>/color/image"로 낸다. -->
+      <plugin filename="ImageDisplay" name="C1 판독 카메라">
         <gz-gui>
-          <property type="double" key="width">380</property>
-          <property type="double" key="height">280</property>
+          <property type="double" key="width">420</property>
+          <property type="double" key="height">320</property>
+          <property type="double" key="z">1</property>
           <property type="string" key="state">floating</property>
+          <property type="bool" key="showTitleBar">true</property>
+          <anchors target="3D View">
+            <line own="right" target="right"/>
+            <line own="top" target="top"/>
+          </anchors>
         </gz-gui>
-        <topic>/c1_conveyor/color</topic>
+        <topic>/c1_conveyor/color/image</topic>
       </plugin>
     </gui>
